Commit message: ggg

File: resources/robots/serialleg/urdf/serialleg.urdf (robot description, URDF)
Before this commit: robot serialleg, 7 links, 6 joints
Joints:
- joint l_wheel_Joint: limit effort=3.0 velocity=49.1.0 -> effort=2.0 velocity=49.1.0
- joint lf0_Joint: limit effort=15.0 velocity=200.0 -> effort=30.0 velocity=200.0
- joint lf1_Joint: limit lower=-0.6 upper=0.8 effort=15.0 velocity=200.0 -> lower=-0.6 upper=0.8 effort=30.0 velocity=200.0
- joint r_wheel_Joint: limit effort=3.0 velocity=49.1 -> effort=2.0 velocity=49.1
- joint rf0_Joint: limit effort=15.0 velocity=200.0 -> effort=30.0 velocity=200.0
- joint rf1_Joint: limit lower=-0.6 upper=0.8 effort=15.0 velocity=200.0 -> lower=-0.6 upper=0.8 effort=30.0 velocity=200.0

Commit message: sim2sim即了

File: resources/robots/serialleg/urdf/serialleg.urdf (robot description, URDF)
Before this commit: robot serialleg, 7 links, 6 joints
Links:
- link base_link: mass 9.8096345 -> 11.88315011

Commit message: 解决网络爆炸

File: resources/robots/serialleg/urdf/serialleg.urdf (robot description, URDF)
Before this commit: robot serialleg, 7 links, 6 joints
Joints:
- joint lf0_Joint: limit effort=30.0 velocity=200.0 -> effort=45.0 velocity=200.0
- joint lf1_Joint: limit lower=-0.6 upper=0.8 effort=30.0 velocity=200.0 -> lower=-0.6 upper=0.8 effort=45.0 velocity=200.0
- joint rf0_Joint: limit effort=30.0 velocity=200.0 -> effort=45.0 velocity=200.0
- joint rf1_Joint: limit lower=-0.6 upper=0.8 effort=30.0 velocity=200.0 -> lower=-0.6 upper=0.8 effort=45.0 velocity=200.0

Commit message: 搞不定气弹簧模拟

File: resources/robots/serialleg/urdf/serialleg.urdf (robot description, URDF)
Before this commit: robot serialleg, 7 links, 6 joints
Links:
- link base_link: mass 9.8096345 -> 11.88315011
Joints:
- joint lf0_Joint: limit effort=30.0 velocity=200.0 -> effort=45.0 velocity=200.0
- joint lf1_Joint: limit lower=-0.6 upper=0.8 effort=30.0 velocity=200.0 -> lower=-0.6 upper=0.8 effort=45.0 velocity=200.0
- joint rf0_Joint: limit effort=30.0 velocity=200.0 -> effort=45.0 velocity=200.0
- joint rf1_Joint: limit lower=-0.6 upper=0.8 effort=30.0 velocity=200.0 -> lower=-0.6 upper=0.8 effort=45.0 velocity=200.0
